File: N22_DCAmplifier/N22_DCAmplifier.kicad_pcb (KiCad board)
At the start: 2 copper layers, 0 parts

Commit message: Updated info, updated N22
Parts:
- added A2201: LF355N, Package_DIP:DIP-8_W7.62mm, F.Cu at (132.7, 96.5)
- added A2202: LF355N, Package_DIP:DIP-8_W7.62mm, F.Cu at (162.0, 114.5)
- added C2201: 470n, Capacitor_THT:C_Rect_L18.0mm_W6.0mm_P15.00mm_FKS3_FKP3, F.Cu at (147.0, 101.5)
- added C2202: 47n/250V, Capacitor_THT:C_Rect_L10.0mm_W4.0mm_P7.50mm_FKS3_FKP3, F.Cu at (174.0, 114.5)
- added C2203: 8p2 / 100V, Capacitor_THT:C_Disc_D4.3mm_W1.9mm_P5.00mm, F.Cu at (173.0, 96.0)
- added C2204: 22u, Capacitor_THT:CP_Radial_Tantal_D4.5mm_P5.00mm, F.Cu at (145.5, 76.5)
- added C2205: 880n, Capacitor_THT:C_Rect_L18.0mm_W5.0mm_P15.00mm_FKS3_FKP3, F.Cu at (140.5, 91.5)
- added C2206: 3n16, Capacitor_THT:C_Axial_L3.8mm_D2.6mm_P15.00mm_Horizontal, F.Cu at (195.0, 101.5)
- added C2207: 6n19 / 63V, Capacitor_THT:C_Axial_L3.8mm_D2.6mm_P15.00mm_Horizontal, F.Cu at (167.5, 104.0)
- added C2209: 22u/10V, Capacitor_THT:C_Disc_D5.0mm_W2.5mm_P5.00mm, F.Cu at (185.5, 109.5)
- added C2210: 33u/10V, Capacitor_THT:CP_Radial_Tantal_D4.5mm_P5.00mm, F.Cu at (153.5, 84.5)
- added C2211: 330n/100V, Capacitor_THT:C_Rect_L18.0mm_W5.0mm_P15.00mm_FKS3_FKP3, F.Cu at (160.0, 89.0)
- added C2212: 4u7/25V, Capacitor_THT:CP_Radial_Tantal_D4.5mm_P5.00mm, F.Cu at (153.5, 73.0)
- added C2213: C_Polarized, Capacitor_THT:C_Disc_D4.7mm_W2.5mm_P5.00mm, F.Cu at (190.0, 109.5)
- added C2216: 27p/100V, Capacitor_THT:C_Disc_D5.1mm_W3.2mm_P5.00mm, F.Cu at (190.0, 107.0)
- added C2217: 3n3/100V, Capacitor_THT:C_Disc_D4.3mm_W1.9mm_P5.00mm, F.Cu at (167.5, 114.5)
- added C2298: C_Polarized, Capacitor_THT:C_Disc_D4.7mm_W2.5mm_P5.00mm, F.Cu at (92.0, 79.0)
- added D2201: HEF4047, Package_DIP:DIP-14_W7.62mm, F.Cu at (192.5, 99.0)
- added JP1: B, TestPoint:TestPoint_Bridge_Pitch2.54mm_Drill1.0mm, F.Cu at (195.0, 117.0)
- added JP2: A, TestPoint:TestPoint_Bridge_Pitch2.54mm_Drill1.0mm, F.Cu at (195.0, 109.8)
- added K1: ~, PM2528:PM2528_RiserCardConnector, F.Cu at (106.1, 121.0)
- added K2201: ~, PM2528:Reed relay assy, F.Cu at (119.5, 76.4)
- added K2202: ~, PM2528:Reed relay assy, F.Cu at (110.5, 114.1)
- added L2201: 470u, Inductor_THT:L_Axial_L9.5mm_D4.0mm_P15.24mm_Horizontal_Fastron_SMCC, F.Cu at (165.0, 114.5)
- added R2201: 681k, Resistor_THT:R_Axial_DIN0207_L6.3mm_D2.5mm_P10.16mm_Horizontal, F.Cu at (148.0, 84.2)
- added R2202: 48k7, Resistor_THT:R_Axial_DIN0207_L6.3mm_D2.5mm_P10.16mm_Horizontal, F.Cu at (170.0, 117.0)
- added R2203: 20k5, Resistor_THT:R_Axial_DIN0207_L6.3mm_D2.5mm_P10.16mm_Horizontal, F.Cu at (115.3, 101.5)
- added R2204: 100k, Resistor_THT:R_Axial_DIN0207_L6.3mm_D2.5mm_P10.16mm_Horizontal, F.Cu at (170.5, 104.0)
- added R2205: 48k7, Resistor_THT:R_Axial_DIN0207_L6.3mm_D2.5mm_P10.16mm_Horizontal, F.Cu at (143.0, 104.5)
- added R2206: 20k5, Resistor_THT:R_Axial_DIN0207_L6.3mm_D2.5mm_P10.16mm_Horizontal, F.Cu at (120.0, 99.1)
- added R2207: 82R5, Resistor_THT:R_Axial_DIN0207_L6.3mm_D2.5mm_P10.16mm_Horizontal, F.Cu at (133.0, 84.5)
- added R2208: 20k5, Resistor_THT:R_Axial_DIN0207_L6.3mm_D2.5mm_P10.16mm_Horizontal, F.Cu at (182.5, 88.7)
- added R2209: 1k, PM2528:Potentiometer horizontal ceramic, F.Cu at (190.5, 73.0)
- added R2210: 1k47, Resistor_THT:R_Axial_DIN0207_L6.3mm_D2.5mm_P10.16mm_Horizontal, F.Cu at (198.0, 104.5)
- added R2211: 1k, Resistor_THT:R_Axial_DIN0207_L6.3mm_D2.5mm_P10.16mm_Horizontal, F.Cu at (135.5, 84.5)
- added R2212: 909, Resistor_THT:R_Axial_DIN0207_L6.3mm_D2.5mm_P10.16mm_Horizontal, F.Cu at (148.0, 116.7)
- added R2213: 220k, Resistor_THT:R_Axial_DIN0207_L6.3mm_D2.5mm_P10.16mm_Horizontal, F.Cu at (177.5, 114.0)
- added R2214: 100, PM2528:Potentiometer horizontal ceramic, F.Cu at (140.5, 70.5)
- added R2215: 9k53, Resistor_THT:R_Axial_DIN0207_L6.3mm_D2.5mm_P10.16mm_Horizontal, F.Cu at (156.0, 84.2)
- added R2216: 47k, PM2528:Potentiometer horizontal ceramic, F.Cu at (198.0, 78.5)
- added R2217: 220k, PM2528:Potentiometer horizontal ceramic, F.Cu at (175.0, 71.0)
- added R2219: 82R5, Resistor_THT:R_Axial_DIN0207_L6.3mm_D2.5mm_P10.16mm_Horizontal, F.Cu at (128.0, 86.5)
- added R2220: 196k, Resistor_THT:R_Axial_DIN0207_L6.3mm_D2.5mm_P10.16mm_Horizontal, F.Cu at (198.0, 91.5)
- added R2221: 48k7, Resistor_THT:R_Axial_DIN0207_L6.3mm_D2.5mm_P10.16mm_Horizontal, F.Cu at (128.0, 107.6)
- added R2222: 1M1, Resistor_THT:R_Axial_DIN0207_L6.3mm_D2.5mm_P10.16mm_Horizontal, F.Cu at (162.0, 104.0)
- added R2223: 20k5, Resistor_THT:R_Axial_DIN0207_L6.3mm_D2.5mm_P10.16mm_Horizontal, F.Cu at (135.5, 116.7)
- added R2224: 20k5, Resistor_THT:R_Axial_DIN0207_L6.3mm_D2.5mm_P10.16mm_Horizontal, F.Cu at (140.5, 116.5)
- added R2225: 196, Resistor_THT:R_Axial_DIN0207_L6.3mm_D2.5mm_P10.16mm_Horizontal, F.Cu at (135.5, 99.1)
- added R2226: 100k, Resistor_THT:R_Axial_DIN0207_L6.3mm_D2.5mm_P10.16mm_Horizontal, F.Cu at (157.0, 104.0)
- added R2227: 100, Resistor_THT:R_Axial_DIN0207_L6.3mm_D2.5mm_P10.16mm_Horizontal, F.Cu at (159.5, 104.0)
- added R2228: 4M7, Resistor_THT:R_Axial_DIN0207_L6.3mm_D2.5mm_P10.16mm_Horizontal, F.Cu at (123.0, 97.0)
- added R2229: 20k5, Resistor_THT:R_Axial_DIN0207_L6.3mm_D2.5mm_P10.16mm_Horizontal, F.Cu at (166.5, 83.5)
- added R2230: 9k09, Resistor_THT:R_Axial_DIN0207_L6.3mm_D2.5mm_P10.16mm_Horizontal, F.Cu at (183.0, 114.0)
- added R2231: 681k, Resistor_THT:R_Axial_DIN0207_L6.3mm_D2.5mm_P10.16mm_Horizontal, F.Cu at (164.0, 83.5)
- added R2232: 100, PM2528:Potentiometer horizontal ceramic, F.Cu at (131.5, 70.5)
- added R2233: 14k7, Resistor_THT:R_Axial_DIN0207_L6.3mm_D2.5mm_P10.16mm_Horizontal, F.Cu at (114.5, 99.0)
- added R2234: 1k96, Resistor_THT:R_Axial_DIN0207_L6.3mm_D2.5mm_P10.16mm_Horizontal, F.Cu at (105.5, 103.6)
- added R2235: 100, Resistor_THT:R_Axial_DIN0207_L6.3mm_D2.5mm_P10.16mm_Horizontal, F.Cu at (130.0, 116.5)
- added R2236: 1k27, Resistor_THT:R_Axial_DIN0207_L6.3mm_D2.5mm_P10.16mm_Horizontal, F.Cu at (192.5, 117.0)
- added R2237: 1k27, Resistor_THT:R_Axial_DIN0207_L6.3mm_D2.5mm_P10.16mm_Horizontal, F.Cu at (198.0, 117.0)
- added R2238: 1M, Resistor_THT:R_Axial_DIN0309_L9.0mm_D3.2mm_P12.70mm_Horizontal, F.Cu at (169.0, 85.8)
- added TP2201: V.Chopper, Connector_Pin:Pin_D0.9mm_L10.0mm_W2.4mm_FlatFork, F.Cu at (192.0, 70.5)
- added TP2202: Demodulator, Connector_Pin:Pin_D0.9mm_L10.0mm_W2.4mm_FlatFork, F.Cu at (161.5, 71.0)
- added TP2203: Chopper Ampl, Connector_Pin:Pin_D0.9mm_L10.0mm_W2.4mm_FlatFork, F.Cu at (157.5, 71.0)
- added TP2204: Hi Out, Connector_Pin:Pin_D0.9mm_L10.0mm_W2.4mm_FlatFork, F.Cu at (117.0, 71.0)
- added TP2205: GND6, Connector_Pin:Pin_D0.9mm_L10.0mm_W2.4mm_FlatFork, F.Cu at (112.0, 71.0)
- added V2201: BFQ10, Package_TO_SOT_THT:TO-75-6, F.Cu at (137.0, 103.5)
- added V2202: BZX79-C4V7, Diode_THT:D_DO-35_SOD27_P10.16mm_Horizontal, F.Cu at (130.5, 76.4)
- added V2203: BAV45, Diode_THT:D_DO-35_SOD27_P5.08mm_Vertical_AnodeUp, F.Cu at (153.0, 104.5)
- added V2204: BAV45, Diode_THT:D_DO-35_SOD27_P5.08mm_Vertical_AnodeUp, F.Cu at (153.0, 96.5)
- added V2205: BSV81, Package_TO_SOT_THT:TO-72-4, F.Cu at (176.5, 97.5)
- added V2206: BC547B, Package_TO_SOT_THT:TO-92_Inline, F.Cu at (145.5, 72.0)
- added V2207: BAW62, Diode_THT:D_DO-35_SOD27_P10.16mm_Horizontal, F.Cu at (143.0, 106.4)
- added V2208: BAW62, Diode_THT:D_DO-35_SOD27_P10.16mm_Horizontal, F.Cu at (145.5, 106.4)
- added V2209: BZX79-C3V6, Diode_THT:D_DO-35_SOD27_P10.16mm_Horizontal, F.Cu at (132.5, 106.4)
- added V2210: BZX79-C3V6, Diode_THT:D_DO-35_SOD27_P10.16mm_Horizontal, F.Cu at (138.0, 106.4)
- added V2211: BZX79-C5V6, Diode_THT:D_DO-35_SOD27_P10.16mm_Horizontal, F.Cu at (179.5, 78.4)
- added V2212: BFW13, Package_TO_SOT_THT:TO-72-4, F.Cu at (173.5, 84.0)
- added V2213: BZX79-C5V1, Diode_THT:D_DO-35_SOD27_P12.70mm_Horizontal, F.Cu at (108.5, 88.7)
- added V2214: BZX79-C5V1, Diode_THT:D_DO-35_SOD27_P12.70mm_Horizontal, F.Cu at (111.5, 88.7)
- added V2215: BAX12A, Diode_THT:D_DO-35_SOD27_P10.16mm_Horizontal, F.Cu at (117.0, 88.8)
Other:
- board outline added: 100.5 x 66.5 mm
- board text added: "ChopperAmpl"
- board text added: "Demod"
- board text added: "Fchop"
- board text added: "GND6"
- board text added: "Gain x10"
- board text added: "HiOut"
- board text added: "Ioff"
- board text added: "SPIKE"
- board text added: "Vchop"
- board text added: "Voff"
