File: N22_DCAmplifier/N22_DCAmplifier.kicad_pcb (KiCad board)
At the start: 2 copper layers, 100.5 x 66.5 mm, 81 parts

Commit message: Small updates, N25 also
Parts:
- moved V2205 0.55 mm to (177.0, 97.3)
Connections:
- R2213 pad 2: Net-(V2205-B) -> Net-(V2205-Bulk)
- R2238 pad 1: Net-(V2205-B) -> Net-(V2205-Bulk)
- V2205 pad 2: Net-(V2205-B) -> Net-(D2201-~{Q})
- V2205 pad 3: Net-(D2201-~{Q}) -> Net-(V2205-Bulk)
- V2205 pad 4: Net-(V2205-B) -> Net-(V2205-Bulk)
