File: N22_DCAmplifier/N22_DCAmplifier.kicad_sch (KiCad schematic)
At the start: 78 parts

Commit message: Updates, add N25
Parts:
- removed JMP1: A, symbol Jumper:Jumper_2_Open
- removed JMP2: B, symbol Jumper:Jumper_2_Open
- added C2298, C2299: C_Polarized, symbol Device:C_Polarized
- added JP1: B, symbol Jumper:Jumper_2_Small_Open
- added JP2: A, symbol Jumper:Jumper_2_Small_Open
- A2201, A2202: value LF355T -> LF355N
- C2204: value 22u/10V -> 22u
- C2206: value 3n16 / 63V -> 3n16
- K1: footprint Philips_PM2528:PM2528_RiserCardConnector -> PM2528:PM2528_RiserCardConnector
- V2203: value BAV15 -> BAV45
- V2204: value BAW45 -> BAV45
- renumbered R2223 to R2233
Connections:
- net 0V is gone; now on net GND5: K1.1 (0V)
- net RELHIGH is gone; now on net RELHI: K2201.1, K2202.1, V2215.2 (A)
- net +15V: now also C2299.1
- net -15V: now also R2230.2, C2298.2; no longer R2230.1
- net GND4: now also JP1.1 (A)
- net GND5: now also UD2201.14 (VDD), C2298.1, C2299.2
- net at C2209.2, UD2201.12 (RETRIGGER), UD2201.8 (+TRIGGER)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: now also R2230.1, UD2201.7 (VSS); no longer R2230.2
- net at R2236.1, R2237.2: now also JP1.2 (B), JP2.1 (A)
- net at R2210.2, R2237.1: now also JP2.2 (B)
- net HIOUT renamed HIOUT1
- net HIOUTADC renamed HIOUT2
Other:
- removed sheet Power
- note added: "-5V, 325Hz"
- note added: "-> ADC (D1101.1, D1101.2) -> Current Source (N23.17)"
- note added: "-> Relays"
- note added: "Chopper"
- note added: "GAIN x10"
- note added: "Ioff"
- note added: "Measuring zero"
- note added: "Power"
- note added: "Supply zero"
- note added: "X1 (Closed) X10 (Open)"
- note removed: "0/-5V, 325Hz"
- note removed: "Choppergen"
- title: N22 DC Amplifier | Main -> Philips PM2528 - N22 (DC Amplifier)
- moved on the sheet: A2202, C2202, C2203, C2206, C2207, C2209, C2210, C2211, C2212, C2216, C2217, K2201B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

Commit message: Updated info, updated N22
Parts:
- added TP2205: GND6, Connector_Pin:Pin_D0.9mm_L10.0mm_W2.4mm_FlatFork, symbol Connector:TestPoint
- A2201, A2202: footprint (none) -> Package_DIP:DIP-8_W7.62mm
- C2201: footprint (none) -> Capacitor_THT:C_Rect_L18.0mm_W6.0mm_P15.00mm_FKS3_FKP3
- C2202: footprint (none) -> Capacitor_THT:C_Rect_L10.0mm_W4.0mm_P7.50mm_FKS3_FKP3
- C2203, C2217: footprint (none) -> Capacitor_THT:C_Disc_D4.3mm_W1.9mm_P5.00mm
- C2204, C2210, C2212: footprint (none) -> Capacitor_THT:CP_Radial_Tantal_D4.5mm_P5.00mm
- C2205, C2211: footprint (none) -> Capacitor_THT:C_Rect_L18.0mm_W5.0mm_P15.00mm_FKS3_FKP3
- C2206, C2207: footprint (none) -> Capacitor_THT:C_Axial_L3.8mm_D2.6mm_P15.00mm_Horizontal
- C2209: footprint (none) -> Capacitor_THT:C_Disc_D5.0mm_W2.5mm_P5.00mm
- C2213: renamed from C2299; footprint (none) -> Capacitor_THT:C_Disc_D4.7mm_W2.5mm_P5.00mm
- C2216: footprint (none) -> Capacitor_THT:C_Disc_D5.1mm_W3.2mm_P5.00mm
- C2298: footprint (none) -> Capacitor_THT:C_Disc_D4.7mm_W2.5mm_P5.00mm
- D2201: renamed from UD2201; footprint (none) -> Package_DIP:DIP-14_W7.62mm
- JP1, JP2: footprint (none) -> TestPoint:TestPoint_Bridge_Pitch2.54mm_Drill1.0mm
- K2201, K2202: footprint (none) -> PM2528:Reed relay assy
- L2201: footprint (none) -> Inductor_THT:L_Axial_L9.5mm_D4.0mm_P15.24mm_Horizontal_Fastron_SMCC
- R2201, R2202, R2203, R2204, R2205, R2206, R2207, R2208, R2210, R2211, R2212, R2213, R2215, R2219, R2220, R2221, R2222, R2223, R2224, R2225, R2226, R2227, R2228, R2229, R2230, R2231, R2233, R2235, R2236, R2237: footprint (none) -> Resistor_THT:R_Axial_DIN0207_L6.3mm_D2.5mm_P10.16mm_Horizontal
- R2209, R2214, R2216, R2217, R2232: footprint (none) -> PM2528:Potentiometer horizontal ceramic
- R2234: value 1k69 -> 1k96; footprint (none) -> Resistor_THT:R_Axial_DIN0207_L6.3mm_D2.5mm_P10.16mm_Horizontal
- R2238: footprint (none) -> Resistor_THT:R_Axial_DIN0309_L9.0mm_D3.2mm_P12.70mm_Horizontal
- TP2201, TP2202, TP2203, TP2204: footprint (none) -> Connector_Pin:Pin_D0.9mm_L10.0mm_W2.4mm_FlatFork
- V2201: footprint (none) -> Package_TO_SOT_THT:TO-75-6
- V2202, V2209, V2210, V2211: footprint (none) -> Diode_THT:D_DO-35_SOD27_P10.16mm_Horizontal
- V2203, V2204: footprint Diode_THT:D_DO-35_SOD27_P7.62mm_Horizontal -> Diode_THT:D_DO-35_SOD27_P5.08mm_Vertical_AnodeUp
- V2205: footprint (none) -> Package_TO_SOT_THT:TO-72-4
- V2207, V2208, V2215: footprint Diode_THT:D_DO-35_SOD27_P7.62mm_Horizontal -> Diode_THT:D_DO-35_SOD27_P10.16mm_Horizontal
- V2212: footprint Package_TO_SOT_THT:TO-92_Inline -> Package_TO_SOT_THT:TO-72-4
- V2213, V2214: footprint (none) -> Diode_THT:D_DO-35_SOD27_P12.70mm_Horizontal
Connections:
- net GND6: now also TP2205.1
- net GND7: now also K2201.6, K2202.6; no longer K2201.2, K2202.2
- net HIOUT1: now also K2201.1; no longer K2201.4
- net HIOUT2: now also K2202.1; no longer K2202.4
- net RELHI: now also K2201.10, K2202.10; no longer K2201.1, K2202.1
Other:
- note added: "(Not fitted)"

Commit message: Started with N24
Other:
- note added: "-> ADC (D1101.1/2) -> Current Source (N23.17)"
- note added: "K2201/K2202: X1 (Closed) X10 (Open)"
- note removed: "(Not fitted)"
- note removed: "-> ADC (D1101.1, D1101.2) -> Current Source (N23.17)"
- note removed: "X1 (Closed) X10 (Open)"
Changed lines of the file:
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@@
 	(title_block
 		(title "Philips PM2528 - N22 (DC Amplifier)")
-		(date "2025-04-08")
+		(date "2025-05-23")
+		(rev "1.1")
 	)
 	(rectangle
@@
 		)
 	)
-	(text "-> ADC (D1101.1, D1101.2)\n-> Current Source (N23.17)\n"
+	(text "-> ADC (D1101.1/2)\n-> Current Source (N23.17)\n"
 		(exclude_from_sim no)
 		(at 204.724 71.12 0)
@@
 		)
 	)
-	(text "X1 (Closed)\nX10 (Open)"
+	(text "K2201/K2202:\nX1 (Closed)\nX10 (Open)"
 		(exclude_from_sim no)
-		(at 162.306 97.536 0)
-		(effects
-			(font
-				(size 1.27 1.27)
-			)
-		)
-	)
-	(text "X1 (Closed)\nX10 (Open)"
-		(exclude_from_sim no)
-		(at 185.928 97.79 0)
-		(effects
-			(font
-				(size 1.27 1.27)
-			)
-		)
-	)
-	(text "(Not fitted)"
-		(exclude_from_sim no)
-		(at 117.856 92.71 0)
+		(at 174.244 99.314 0)
 		(effects
 			(font
@@
 	(wire
 		(pts
-			(xy 223.52 214.63) (xy 223.52 215.9)
+			(xy 223.52 214.63) (xy 223.52 218.44)
 		)
 		(stroke
@@
 	(symbol
 		(lib_id "power:GND3")
-		(at 223.52 215.9 0)
+		(at 223.52 218.44 0)
 		(unit 1)
 		(exclude_from_sim no)
@@
 		(dnp no)
 		(property "Reference" "#PWR021"
-			(at 223.52 222.25 0)
+			(at 223.52 224.79 0)
 			(effects
 				(font
@@
 		)
 		(property "Value" "GND4"
-			(at 223.52 219.71 0)
+			(at 223.52 222.25 0)
 			(effects
 				(font
@@
 		)
 		(property "Footprint" ""
-			(at 223.52 215.9 0)
+			(at 223.52 218.44 0)
 			(effects
 				(font
@@
 		)
 		(property "Datasheet" ""
-			(at 223.52 215.9 0)
+			(at 223.52 218.44 0)
 			(effects
 				(font
@@
 		)
 		(property "Description" "Power symbol creates a global label with name \"GND3\" , ground"
-			(at 223.52 215.9 0)
+			(at 223.52 218.44 0)
 			(effects
 				(font

Commit message: Small updates, N25 also
Parts:
- removed V2205: BSV81, Package_TO_SOT_THT:TO-72-4, symbol PM2528:BVS81
- added V2205: BSV81, Package_TO_SOT_THT:TO-72-4, symbol Simulation_SPICE:NMOS_Substrate
Connections:
- net at C2203.2, C2207.1, R2204.2: now also V2205.1 (D)
- net at D2201.11 (~{Q}), TP2201.1: now also V2205.2 (G)
- net at R2213.2, R2238.1: now also V2205.3 (S), V2205.4 (Bulk)
Changed lines of the file:
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@@
 	)
 	(junction
-		(at 127 246.38)
-		(diameter 0)
-		(color 0 0 0 0)
-	)
-	(junction
 		(at 372.11 215.9)
 		(diameter 0)
@@
 	)
 	(junction
+		(at 139.7 179.07)
+		(diameter 0)
+		(color 0 0 0 0)
+	)
+	(junction
 		(at 85.09 209.55)
 		(diameter 0)
@@
 	)
 	(junction
-		(at 139.7 179.07)
-		(diameter 0)
-		(color 0 0 0 0)
-	)
-	(junction
 		(at 142.24 71.12)
 		(diameter 0)
@@
 	)
 	(junction
+		(at 128.27 246.38)
+		(diameter 0)
+		(color 0 0 0 0)
+	)
+	(junction
 		(at 172.72 151.13)
 		(diameter 0)
@@
 	(wire
 		(pts
-			(xy 127 186.69) (xy 127 246.38)
+			(xy 128.27 185.42) (xy 128.27 246.38)
 		)
 		(stroke
@@
 	(wire
 		(pts
+			(xy 139.7 179.07) (xy 139.7 180.34)
+		)
+		(stroke
+			(width 0)
+			(type default)
+		)
+	)
+	(wire
+		(pts
 			(xy 90.17 261.62) (xy 92.71 261.62)
 		)
@@
 	(wire
 		(pts
-			(xy 123.19 246.38) (xy 127 246.38)
+			(xy 123.19 246.38) (xy 128.27 246.38)
 		)
 		(stroke
@@
 	(wire
 		(pts
+			(xy 128.27 246.38) (xy 133.35 246.38)
+		)
+		(stroke
+			(width 0)
+			(type default)
+		)
+	)
+	(wire
+		(pts
 			(xy 93.98 27.94) (xy 93.98 29.21)
 		)
@@
 	(wire
 		(pts
-			(xy 139.7 180.34) (xy 139.7 179.07)
-		)
-		(stroke
-			(width 0)
-			(type default)
-		)
-	)
-	(wire
-		(pts
 			(xy 388.62 215.9) (xy 388.62 217.17)
 		)
@@
 	(wire
 		(pts
+			(xy 139.7 179.07) (xy 154.94 179.07)
+		)
+		(stroke
+			(width 0)
+			(type default)
+		)
+	)
+	(wire
+		(pts
 			(xy 166.37 92.71) (xy 166.37 93.98)
 		)
@@
 	(wire
 		(pts
-			(xy 139.7 179.07) (xy 154.94 179.07)
-		)
-		(stroke
-			(width 0)
-			(type default)
-		)
-	)
-	(wire
-		(pts
 			(xy 350.52 44.45) (xy 350.52 45.72)
 		)
@@
 	(wire
 		(pts
-			(xy 127 246.38) (xy 133.35 246.38)
-		)
-		(stroke
-			(width 0)
-			(type default)
-		)
-	)
-	(wire
-		(pts
 			(xy 95.25 209.55) (xy 93.98 209.55)
 		)
@@
 	(wire
 		(pts
-			(xy 127 186.69) (xy 132.08 186.69)
+			(xy 128.27 185.42) (xy 133.35 185.42)
 		)
 		(stroke
@@
 	)
 	(symbol
+		(lib_id "Simulation_SPICE:NMOS_Substrate")
+		(at 137.16 185.42 0)
+		(unit 1)
+		(exclude_from_sim no)
+		(in_bom yes)
+		(on_board yes)
+		(dnp no)
+		(property "Reference" "V2205"
+			(at 143.256 181.864 0)
+			(effects
+				(font
+					(size 1.27 1.27)
+				)
+				(justify left)
+			)
+		)
+		(property "Value" "BSV81"
+			(at 143.51 183.896 0)
+			(effects
+				(font
+					(size 1.27 1.27)
+				)
+				(justify left)
+			)
+		)
+		(property "Footprint" "Package_TO_SOT_THT:TO-72-4"
+			(at 167.005 185.42 0)
+			(effects
+				(font
+					(size 1.27 1.27)
+				)
+				(hide yes)
+			)
+		)
+		(property "Datasheet" "https://ngspice.sourceforge.io/docs/ngspice-html-manual/manual.xhtml#cha_MOSFETs"
+			(at 137.16 204.47 0)
+			(effects
+				(font
+					(size 1.27 1.27)
+				)
+				(hide yes)
+			)
+		)
+		(property "Description" "N-channel MOSFET symbol with substrate (bulk) pin"
+			(at 137.16 185.42 0)
+			(effects
+				(font
+					(size 1.27 1.27)
+				)
+				(hide yes)
+			)
+		)
+		(property "Sim.Device" "NMOS"
+			(at 137.16 201.93 0)
+			(effects
+				(font
+					(size 1.27 1.27)
+				)
+				(hide yes)
+			)
+		)
+		(property "Sim.Type" "MOS1"
+			(at 137.16 200.025 0)
+			(effects
+				(font
+					(size 1.27 1.27)
+				)
+				(hide yes)
+			)
+		)
+		(property "Sim.Pins" "1=D 2=G 3=S 4=B"
+			(at 137.16 198.12 0)
+			(effects
+				(font
+					(size 1.27 1.27)
+				)
+				(hide yes)
+			)
+		)
+		(pin "3"
+		)
+		(pin "1"
+		)
+		(pin "2"
+		)
+		(pin "4"
+		)
+		(instances
+			(project ""
+				(path "/2ba4ca6b-4aec-411c-9da4-218d92fedde9"
+					(reference "V2205")
+					(unit 1)
+				)
+			)
+		)
+	)
+	(symbol
 		(lib_id "Diode:BAW75")
 		(at 72.39 29.21 180)
@@
 					(unit 1)
 				)
-			)
-		)
-	)
-	(symbol
-		(lib_id "PM2528:BVS81")
-		(at 138.43 185.42 0)
-		(unit 1)
-		(exclude_from_sim no)
-		(in_bom yes)
-		(on_board yes)
-		(dnp no)
-		(property "Reference" "V2205"
-			(at 141.478 182.372 0)
-			(effects
-				(font
-					(size 1.27 1.27)
-				)
-				(justify left)
-			)
-		)
-		(property "Value" "BSV81"
-			(at 141.478 184.15 0)
-			(effects
-				(font
-					(size 1.27 1.27)
-				)
-				(justify left)
-			)
-		)
-		(property "Footprint" "Package_TO_SOT_THT:TO-72-4"
-			(at 138.43 185.42 0)
-			(effects
-				(font
-					(size 1.27 1.27)
-				)
-				(hide yes)
-			)
-		)
-		(property "Datasheet" ""
-			(at 138.43 185.42 0)
-			(effects
-				(font
-					(size 1.27 1.27)
-				)
-				(hide yes)
-			)
-		)
-		(property "Description" ""
-			(at 138.43 185.42 0)
-			(effects
-				(font
-					(size 1.27 1.27)
-				)
-				(hide yes)
-			)
-		)
-		(pin "2"
-		)
-		(pin "4"
-		)
-		(pin "3"
-		)
-		(pin "1"
-		)
-		(instances
-			(project ""
-				(path "/2ba4ca6b-4aec-411c-9da4-218d92fedde9"
-					(reference "V2205")
-					(unit 1)
-				)
