File: N25_RMSConverter/N25_RMSConverter.kicad_pcb (KiCad board)
At the start: 2 copper layers, 100.5 x 64.5 mm, 26 parts

Commit message: N25 RMS Ok!
Parts:
- added C2501: 22p, Capacitor_THT:C_Disc_D4.3mm_W1.9mm_P5.00mm, F.Cu at (171.5, 93.5)
- added C2502: 470p, Capacitor_THT:C_Disc_D4.3mm_W1.9mm_P5.00mm, F.Cu at (175.5, 78.0)
- added C2503: 100p, Capacitor_THT:C_Disc_D4.3mm_W1.9mm_P5.00mm, F.Cu at (160.0, 111.5)
- added C2504: 10n, Capacitor_THT:C_Disc_D4.3mm_W1.9mm_P5.00mm, F.Cu at (165.5, 112.0)
- added C2505: 10n, Capacitor_THT:C_Disc_D4.3mm_W1.9mm_P5.00mm, F.Cu at (167.5, 114.5)
- added C2506: 3u3, Capacitor_THT:C_Rect_L26.5mm_W8.5mm_P22.50mm_MKS4, F.Cu at (124.0, 109.0)
- added C2507: 330n, Capacitor_THT:C_Rect_L18.0mm_W5.0mm_P15.00mm_FKS3_FKP3, F.Cu at (132.0, 96.0)
- added C2508: 10p, Capacitor_THT:C_Disc_D4.3mm_W1.9mm_P5.00mm, F.Cu at (142.5, 101.5)
- added C2509: 100p, Capacitor_THT:C_Disc_D4.3mm_W1.9mm_P5.00mm, F.Cu at (134.0, 114.0)
- added C2510: 470p, Capacitor_THT:C_Disc_D4.3mm_W1.9mm_P5.00mm, F.Cu at (152.0, 114.5)
- added C2511: 6u8, Capacitor_THT:CP_Radial_Tantal_D7.0mm_P5.00mm, F.Cu at (187.5, 109.0)
- added C2512: 6u8, Capacitor_THT:CP_Radial_Tantal_D7.0mm_P5.00mm, F.Cu at (178.5, 109.0)
- added C2513: 22n, Capacitor_THT:C_Disc_D4.3mm_W1.9mm_P5.00mm, F.Cu at (183.0, 114.0)
- added C2514: 22n, Capacitor_THT:C_Disc_D4.3mm_W1.9mm_P5.00mm, F.Cu at (187.0, 104.5)
- added C2515: 6u8, Capacitor_THT:C_Rect_L31.5mm_W13.0mm_P27.50mm_MKS4, F.Cu at (103.0, 108.8)
- added C2516: 2u2, Capacitor_THT:C_Rect_L26.5mm_W8.5mm_P22.50mm_MKS4, F.Cu at (114.5, 108.8)
- added C2517: 100n, Capacitor_THT:C_Rect_L13.0mm_W4.0mm_P10.00mm_FKS3_FKP3_MKS4, F.Cu at (125.5, 81.5)
- added C2518: 10n, Capacitor_THT:C_Disc_D4.3mm_W1.9mm_P5.00mm, F.Cu at (167.5, 98.5)
- added C2519: 2n2, Capacitor_THT:C_Disc_D4.3mm_W1.9mm_P5.00mm, F.Cu at (167.5, 96.0)
- added C2520: 18p, Capacitor_THT:C_Disc_D4.3mm_W1.9mm_P5.00mm, F.Cu at (162.5, 100.0)
- added R2502: 19R6, Resistor_THT:R_Axial_DIN0207_L6.3mm_D2.5mm_P10.16mm_Horizontal, F.Cu at (182.0, 106.0)
- added R2503: 301k, Resistor_THT:R_Axial_DIN0207_L6.3mm_D2.5mm_P10.16mm_Horizontal, F.Cu at (184.5, 106.0)
- added R2505: 750, Resistor_THT:R_Axial_DIN0207_L6.3mm_D2.5mm_P10.16mm_Horizontal, F.Cu at (183.0, 93.5)
- added R2506: 590, Resistor_THT:R_Axial_DIN0207_L6.3mm_D2.5mm_P10.16mm_Horizontal, F.Cu at (180.5, 91.0)
- added R2507: 301, Resistor_THT:R_Axial_DIN0207_L6.3mm_D2.5mm_P10.16mm_Horizontal, F.Cu at (188.5, 86.0)
- added R2508: 7k87, Resistor_THT:R_Axial_DIN0207_L6.3mm_D2.5mm_P10.16mm_Horizontal, F.Cu at (188.0, 98.5)
- added R2509: 1k96, Resistor_THT:R_Axial_DIN0207_L6.3mm_D2.5mm_P10.16mm_Horizontal, F.Cu at (185.5, 93.5)
- added R2511: 8R25, Resistor_THT:R_Axial_DIN0207_L6.3mm_D2.5mm_P10.16mm_Horizontal, F.Cu at (168.0, 80.5)
- added R2512: 115, Resistor_THT:R_Axial_DIN0207_L6.3mm_D2.5mm_P10.16mm_Horizontal, F.Cu at (179.0, 105.0)
- added R2513: 301k, Resistor_THT:R_Axial_DIN0207_L6.3mm_D2.5mm_P10.16mm_Horizontal, F.Cu at (165.0, 82.5)
- added R2515: 2k05, Resistor_THT:R_Axial_DIN0207_L6.3mm_D2.5mm_P10.16mm_Horizontal, F.Cu at (162.5, 112.5)
- added R2516: 4k02, Resistor_THT:R_Axial_DIN0207_L6.3mm_D2.5mm_P10.16mm_Horizontal, F.Cu at (149.0, 114.5)
- added R2520: 5M6, Resistor_THT:R_Axial_DIN0207_L6.3mm_D2.5mm_P10.16mm_Horizontal, F.Cu at (168.0, 93.5)
- added R2521: 33M, Resistor_THT:R_Axial_DIN0207_L6.3mm_D2.5mm_P10.16mm_Horizontal, F.Cu at (175.5, 108.7)
- added S2501: SW_DPST_x2, Button_Switch_THT:SW_DIP_SPSTx02_Slide_6.7x6.64mm_W7.62mm_P2.54mm_LowProfile, F.Cu at (99.9, 66.5)
- added V2501: BC547B, Package_TO_SOT_THT:TO-92, F.Cu at (180.0, 74.5)
- added V2502: BC547B, Package_TO_SOT_THT:TO-92, F.Cu at (185.5, 75.0)
- added V2503: BC559B, Package_TO_SOT_THT:TO-92, F.Cu at (185.5, 80.5)
- added V2508: BAW62, Diode_THT:D_DO-34_SOD68_P10.16mm_Horizontal, F.Cu at (170.5, 69.8)
- added V2509: BAW62, Diode_THT:D_DO-34_SOD68_P10.16mm_Horizontal, F.Cu at (173.5, 80.0)
- added V2510: BZX79-B4V7, Diode_THT:D_DO-34_SOD68_P10.16mm_Horizontal, F.Cu at (165.0, 87.0)
- added V2511: BAV45, Package_TO_SOT_THT:TO-18-2, F.Cu at (160.5, 92.5)
- added V2512: BAV45, Package_TO_SOT_THT:TO-18-2, F.Cu at (135.5, 106.0)
- added V2513: BAW62, Diode_THT:D_DO-34_SOD68_P10.16mm_Horizontal, F.Cu at (136.4, 114.5)
- added V2514: BAV45, Package_TO_SOT_THT:TO-18-2, F.Cu at (107.5, 77.0)
- added V2515: BAX12A, Diode_THT:D_DO-34_SOD68_P10.16mm_Horizontal, F.Cu at (136.5, 70.4)
- R2501: value ~ -> OM529
- moved TP2506 38.0 mm to (137.0, 84.0)
- moved R2518 4.95 mm to (131.0, 114.6)
- moved R2519 3.64 mm to (128.0, 113.0), turned to 180 degrees
- moved V2504 3.20 mm to (149.2, 89.2)
- moved A2503 2.00 mm to (145.0, 98.5)
- moved R2501 0.38 mm to (162.0, 76.0)
Connections:
- JP2 pad 1: Net-(JP1-B) -> Net-(JP2-A)
- JP3 pad 1: Net-(JP2-B) -> Net-(JP3-A)
- JP4 pad 1: Net-(JP3-B) -> Net-(JP4-A)
- R2501 pad 4: Net-(JP1-A) -> Net-(JP1-B)
- R2501 pad 5: Net-(JP1-B) -> Net-(JP1-A)
- R2501 pad 6: Net-(JP2-B) -> Net-(JP2-A)
- R2501 pad 7: Net-(JP3-B) -> Net-(JP3-A)
- R2501 pad 8: Net-(JP4-B) -> Net-(JP4-A)
- R2517 pad 3: Net-(JP4-B) -> Net-(JP4-A)
