File: N25_RMSConverter/N25_RMSConverter.kicad_sch (KiCad schematic)
At the start: 72 parts

Commit message: Small updates, N25 also
Parts:
- A2502: footprint Package_SO:SOIC-8_3.9x4.9mm_P1.27mm -> Package_DIP:DIP-8_W7.62mm
- JP1, JP2, JP3, JP4: footprint (none) -> TestPoint:TestPoint_Bridge_Pitch5.08mm_Drill0.7mm
- K2515: footprint (none) -> PM2528:Reed relay assy
- R2504, R2510, R2514, R2517: footprint (none) -> PM2528:Potentiometer horizontal ceramic
- R2518, R2519: footprint (none) -> Resistor_THT:R_Axial_DIN0207_L6.3mm_D2.5mm_P10.16mm_Horizontal
- TP2501, TP2502, TP2503, TP2504, TP2505, TP2506, TP2507: footprint (none) -> Connector_PinHeader_1.00mm:PinHeader_1x01_P1.00mm_Vertical
- renumbered D2506 to D2508
Connections:
- net D1703.22: now also K2515.10; no longer K2515.1
- net GND6: now also K2515.6; no longer K2515.2
- net at R2501.9: now also K2515.1; no longer K2515.4
Other:
- note added: "DC Level at Vin=+1V"
- moved on the sheet: C2518, C2519, R2520, R2521, TP2505

Commit message: N25 RMS Ok!
Parts:
- C2501, C2502, C2504, C2505, C2508, C2509, C2510, C2513, C2514, C2518, C2519: footprint (none) -> Capacitor_THT:C_Disc_D4.3mm_W1.9mm_P5.00mm
- C2503: value 82p -> 100p; footprint (none) -> Capacitor_THT:C_Disc_D4.3mm_W1.9mm_P5.00mm
- C2506, C2516: footprint (none) -> Capacitor_THT:C_Rect_L26.5mm_W8.5mm_P22.50mm_MKS4
- C2507: footprint (none) -> Capacitor_THT:C_Rect_L18.0mm_W5.0mm_P15.00mm_FKS3_FKP3
- C2511: renamed from C2533; footprint (none) -> Capacitor_THT:CP_Radial_Tantal_D7.0mm_P5.00mm
- C2512: renamed from C2534; footprint (none) -> Capacitor_THT:CP_Radial_Tantal_D7.0mm_P5.00mm
- C2515: footprint (none) -> Capacitor_THT:C_Rect_L31.5mm_W13.0mm_P27.50mm_MKS4
- C2517: footprint (none) -> Capacitor_THT:C_Rect_L13.0mm_W4.0mm_P10.00mm_FKS3_FKP3_MKS4
- C2520: value 15p -> 18p; footprint (none) -> Capacitor_THT:C_Disc_D4.3mm_W1.9mm_P5.00mm
- R2501: value ~ -> OM529
- R2502, R2503, R2505, R2506, R2507, R2508, R2509, R2511, R2512, R2513, R2515, R2516, R2520, R2521: footprint (none) -> Resistor_THT:R_Axial_DIN0207_L6.3mm_D2.5mm_P10.16mm_Horizontal
- S2501: footprint (none) -> Button_Switch_THT:SW_DIP_SPSTx02_Slide_6.7x6.64mm_W7.62mm_P2.54mm_LowProfile
- V2501, V2502, V2503: footprint (none) -> Package_TO_SOT_THT:TO-92
- V2508: renamed from D2508; footprint (none) -> Diode_THT:D_DO-34_SOD68_P10.16mm_Horizontal
- V2509: renamed from D2509; footprint (none) -> Diode_THT:D_DO-34_SOD68_P10.16mm_Horizontal
- V2510: value BZX79-C4V7 -> BZX79-B4V7; footprint (none) -> Diode_THT:D_DO-34_SOD68_P10.16mm_Horizontal
- V2511: renamed from D2511; footprint (none) -> Package_TO_SOT_THT:TO-18-2
- V2512, V2514: footprint (none) -> Package_TO_SOT_THT:TO-18-2
- V2513, V2515: footprint (none) -> Diode_THT:D_DO-34_SOD68_P10.16mm_Horizontal
Connections:
- net at JP1.1 (A): now also JP2.2 (B), R2501.5; no longer R2501.4
- net at R2501.8, R2517.3: now also JP4.1 (A); no longer JP4.2 (B)
- new net: JP1.2 (B), R2501.4
- new net: JP3.1 (A), JP4.2 (B), R2501.7
- new net: JP2.1 (A), JP3.2 (B), R2501.6
Other:
- note added: "DC Level at Vin= ≈1V RMS"
- note removed: "DC Level at Vin=+1V"
- moved on the sheet: C2515, C2516, C2517, C2519, K2515B, R2510, R2511, R2517, R2518, R2519, R2521, S2501B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
