File: Schematics/N20_ADCControl/N20_ADCControl.kicad_pcb (KiCad board)
At the start: 2 copper layers, 96.5 x 62 mm, 36 parts

Commit message: Lotsofchanges. Included Ghidra-project and correct firmware-images
Parts:
- K1: footprint Philips_PM2528:PM2528_RiserCardConnector -> PM2528:PM2528_RiserCardConnector
- TP2001, TP2002, TP2003, TP2004, TP2005, TP2006, TP2007, TP2008, TP2009, TP2010, TP2011, TP2012, TP2013: footprint Connector_PinHeader_1.00mm:PinHeader_1x01_P1.00mm_Vertical -> Connector_Pin:Pin_D1.0mm_L10.0mm
Connections:
- net /SCP renamed /_SCP
