File: Schematics/N22_DCAmplifier/N22_DCAmplifier.kicad_sch (KiCad schematic)
At the start: 81 parts

Commit message: Lotsofchanges. Included Ghidra-project and correct firmware-images
Other:
- note added: "-> ADC -> Currentsource.Filter (N23)"
- note removed: "-> ADC (D1101.1/2) -> Current Source (N23.17)"
Changed lines of the file:
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@@
 	)
 	(rectangle
-		(start 50.8 166.37)
+		(start 46.99 166.37)
 		(end 247.65 215.9)
 		(stroke
@@
 	)
 	(rectangle
-		(start 50.8 218.44)
+		(start 46.99 218.44)
 		(end 144.78 281.94)
 		(stroke
@@
 		)
 	)
-	(text "-> ADC (D1101.1/2)\n-> Current Source (N23.17)\n"
+	(text "-> ADC\n-> Currentsource.Filter (N23)\n"
 		(exclude_from_sim no)
 		(at 204.724 71.12 0)
@@
 	(text "DC"
 		(exclude_from_sim no)
-		(at 53.848 169.418 0)
+		(at 49.53 168.656 0)
 		(effects
 			(font
@@
 	(text "Chopper"
 		(exclude_from_sim no)
-		(at 58.42 220.726 0)
+		(at 52.324 220.726 0)
 		(effects
 			(font
@@
 	)
 	(hierarchical_label "LO"
-		(shape input)
+		(shape output)
 		(at 29.21 43.18 0)
 		(effects
@@
 					(size 1.27 1.27)
 				)
+				(hide yes)
 			)
 		)
@@
 					(size 1.27 1.27)
 				)
+				(hide yes)
 			)
 		)
@@
 					(size 1.27 1.27)
 				)
+				(hide yes)
 			)
 		)
@@
 					(size 1.27 1.27)
 				)
+				(hide yes)
 			)
 		)
@@
 					(size 1.27 1.27)
 				)
+				(hide yes)
 			)
 		)
@@
 					(size 1.27 1.27)
 				)
+				(hide yes)
 			)
 		)
