File: Schematics/ExpensionCards/N30_GalvanicSeperation/N30_GalvanicSeperation.kicad_sch (KiCad schematic)
At the start: 46 parts, among them X3010 Conn_01x01_MountingPin, X3011 Conn_01x01_MountingPin, X3012 Conn_01x01_MountingPin

Commit message: Updated disassembly some more Moved PM2528 footprints/3D to subfolder
Parts:
- X3001: footprint PM2528:PM2528_RiserCardConnector -> Philips_PM2528:PM2528_RiserCardConnector
Changed lines of the file:
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@@
 	(title_block
 		(title "Philips PM2528 - N30 (Galvanic Seperation)")
-		(date "2025-08-17")
+		(date "2025-08-23")
 		(rev "1.0")
 		(company "D. Kupers")
@@
 			)
 		)
-		(property "Footprint" "PM2528:PM2528_RiserCardConnector"
+		(property "Footprint" "Philips_PM2528:PM2528_RiserCardConnector"
 			(at 36.83 24.13 0)
 			(effects
